File: CAD/Tools/PCB_Reflow/Reflow_Heater/Reflow_Heater.sch (KiCad schematic (older format))
At the start: 6 parts, among them J1 Screw Connector, J2 Screw_Connector

Commit message: feat: 100x50 (78x49 usable space) smaller heater & gerbers
Parts:
- added MH5: ThermalFuse, Mounting_Holes:MountingHole_3.2mm_M3, symbol Mechanical:MountingHole
Changed lines of the file:
@@
 Wire Wire Line
 	2700 1400 2300 1400
+$Comp
+L Mechanical:MountingHole MH5
+U 1 1 61FD9CBE
+P 1000 1900
+F 0 "MH5" H 1100 1946 50  0000 L CNN
+F 1 "ThermalFuse" H 1100 1855 50  0000 L CNN
+F 2 "Mounting_Holes:MountingHole_3.2mm_M3" H 1000 1900 50  0001 C CNN
+F 3 "~" H 1000 1900 50  0001 C CNN
+	1    1000 1900
+	1    0    0    -1
+$EndComp
 $EndSCHEMATC
